File: voltage_board.kicad_sch (KiCad schematic)
At the start: 14 parts, among them J1 USB4105GFA060, U1 MAX77654AENV+T

Commit message: schematic finished
Parts:
- removed C1: 4.7uF, passive:0603, symbol passive:capacitor_0805
- removed C2: 1uF, passive:0402, symbol passive:capacitor_0805
- removed C3, C6: 22uF, passive:0603, symbol passive:capacitor_0603
- removed C5: 4.7uF, passive:0603, symbol passive:capacitor_0603
- added C1, C10, C2, C3, C4: 22uF, passive:0402, symbol passive:capacitor_0402
- added C11, C13, C14, C8: 1uF, passive:0402, symbol passive:capacitor_0402
- added C12, C9: 4.7uF, passive:0402, symbol passive:capacitor_0402
- added C6, C7: 2.2uF, passive:0402, symbol passive:capacitor_0402
- added J2: 53261-0271, connector:53261-0271, symbol connector:53261-0271
- added R1, R2: 0R, passive:0402, symbol passive:resistor_0402
- added R10: 100K, passive:0402, symbol passive:resistor_0402
- added R8, R9: 10K, passive:0402, symbol passive:resistor_0402
- added RT1: NTCLE413E2103H400, passive:THT2, symbol passive:thermal_resistor_tht
- added S1: TL3365AF180QG, connector:TL3365AF180QG, symbol connector:TL3365AF180QG
- U1: footprint power:BGA30C40P6X5_279X234X50 -> BGA30C40P6X5_279X234X50
- renumbered C4 to C5, R5 to R3, R1 to R4, R2 to R5, R3 to R6, R4 to R7
Connections:
- net BATT: now also C10.1, C9.2, J2.1
- net CHGIN: now also C12.2
- net GND: now also U1.C3 (GND), C1.2, C10.2, C11.2, C12.1, C13.2, C14.2, C2.2, C3.2, C4.2, C6.2, C7.2, C8.2, C9.1, J2.2, J2.MP1, J2.MP2, RT1.2, S1.1, S1.2
- net VL: now also U1.D1 (VL), C13.1
- net at R3.1, U1.E4 (IN_SBB): now also C4.1
- net GPIO1: now reaches U1.A1 (GPIO1)
- net nRST: now reaches U1.A2 (nRST)
- net nRST: now also R9.1
- net VIO: now reaches U1.A4 (VIO)
- net VIO: now also C14.1, R10.1, R9.2
- net LDO1: now reaches U1.A5 (LDO1)
- net LDO1: now also C11.1
- net IN_LDO1: now reaches U1.A6 (IN_LDO1)
- net IN_LDO1: now also C7.1, R1.2
- net GPIO0: now reaches U1.B1 (GPIO0)
- net nIRQ: now reaches U1.B2 (nIRQ)
- net nIRQ: now also R10.2
- net nEN: now reaches U1.B3 (nEN)
- net nEN: now also S1.3, S1.4
- net LDO0: now reaches U1.B5 (LDO0)
- net LDO0: now also C8.1
- net IN_LDO0: now reaches U1.B6 (IN_LDO0)
- net IN_LDO0: now also C6.1, R2.2
- net AMUX: now reaches U1.C1 (AMUX)
- net GPIO2: now reaches U1.C2 (GPIO2)
- net SSB1: now reaches U1.C4 (SBB1)
- net SSB1: now also C1.1
- net SSB0: now reaches U1.C6 (SBB0)
- net SSB0: now also C2.1, R1.1, R2.1
- net THM: now reaches U1.D2 (THM)
- net THM: now also R8.1, RT1.1
- net TBIAS: now reaches U1.D3 (TBIAS)
- net TBIAS: now also R8.2
- net SSB2: now reaches U1.D4 (SBB2)
- net SSB2: now also C3.1
Other:
- note added: "Before connecting the battery to the board, make sure the polarity matches."
- moved on the sheet: R3, U1

Commit message: layout almost finished
Parts:
- removed C6, C7: 2.2uF, passive:0402, symbol passive:capacitor_0402
- removed R1, R2, R3: 0R, passive:0402, symbol passive:resistor_0402
- added C15: 22uF, passive:0402, symbol passive:capacitor_0402
- C4: footprint passive:0402 -> passive:0603; symbol passive:capacitor_0402 -> passive:capacitor_0603
Connections:
- net IN_LDO0 is gone; now on net SSB0: U1.B6 (IN_LDO0)
- net IN_LDO1 is gone; now on net SSB0: U1.A6 (IN_LDO1)
- net GND: now also C15.2
- net V_SYS: now also C4.1, U1.E4 (IN_SBB), C15.1

Commit message: almost done the PCB
Connections:
- net SDA: now reaches U1.A3 (SDA)
- net SCL: now reaches U1.B4 (SCL)
Changed lines of the file:
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@@
     (effects (font (size 1.27 1.27)) (justify left bottom))
+  )
+  (label "SDA" (at 35.56 154.94 180) (fields_autoplaced)
+    (effects (font (size 1.27 1.27)) (justify right bottom))
   )
   (label "USB_CC1" (at 68.58 25.4 0) (fields_autoplaced)
@@
     (effects (font (size 1.27 1.27)) (justify left bottom))
   )
+  (label "SCL" (at 35.56 172.72 180) (fields_autoplaced)
+    (effects (font (size 1.27 1.27)) (justify right bottom))
+  )
   (label "USB_DN" (at 68.58 30.48 0) (fields_autoplaced)

Commit message: backup
Parts:
- removed R6, R7: 27R, passive:0402, symbol passive:resistor_0402
- added J4: ~, connector:Connector_20PIN_5052782033, symbol connector:Connector_20PIN_5052782033
Connections:
- net CHGIN: now also J4.19, J4.20
- net GND: now also J4.1, J4.11, J4.17, J4.18, J4.3, J4.5, J4.7, J4.9
- net LDO0: now also J4.8
- net LDO1: now also J4.10
- net SCL: now also J4.12
- net SDA: now also J4.13
- net SSB0: now also J4.6
- net SSB1: now also J4.4
- net SSB2: now also J4.2
- net USB_DN: no longer J1.A7 (DN1)
- net USB_DP: no longer J1.A6 (DP1)
- net nEN: now also J4.15
- net nIRQ: now also J4.16
- net nRST: now also J4.14

Commit message: done ;).
Parts:
- removed C11, C8: 1uF, passive:0402, symbol passive:capacitor_0402
- added C6, C7: 1uF, passive:C_0402, symbol passive:capacitor_0402
- added J3: ~, connector:Header_THT_1.27_3P, symbol connector:Header_1.27_3PIN
- C1, C10, C12, C13, C14, C15, C2, C3, C5, C9: footprint passive:0402 -> passive:C_0402
- C4: footprint passive:0603 -> passive:C_0603
- L1: footprint passive:2016 -> passive:L_0806; symbol passive:inductor_2016 -> passive:inductor_0806
- R10, R4, R5, R8, R9: footprint passive:0402 -> passive:R_0402
Connections:
- net AMUX: now also J3.3
- net GND: now also C6.2, C7.2
- net GPIO0: now also J3.2
- net GPIO1: now also J3.1
- net LDO0: now also C6.1
- net LDO1: now also C7.1
- net SSB0: now also C3.1; no longer C2.1
- net SSB1: now also C2.1; no longer C1.1
- net SSB2: now also C1.1; no longer C3.1
- net GPIO2: no longer names the net of U1.C2 (GPIO2)
- net USB_CC1: no longer names the net of J1.B5 (CC2), R4.2
- net USB_CC2: no longer names the net of J1.A5 (CC1), R5.2
- net USB_DN: no longer names the net of J1.B7 (DN2)
- net USB_DP: no longer names the net of J1.B6 (DP2)
- no-connect marks 0 -> 7
Other:
- note added: "Battery Connector"
- note added: "On/Off Button"
- note added: "Output Connector"
- note added: "Power Management Core"
- note added: "TEST Points"
- note added: "USB-C Connector"
- moved on the sheet: C1, C10, C12, C13, C14, C15, C2, C3, C4, C5, C9, J1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
