File: voltage_board.kicad_pcb (KiCad board)
At the start: 4 copper layers, 50.8 x 50.8 mm, 14 parts, among them J1 USB4105GFA060, U1 MAX77654AENV+T

Commit message: schematic finished
Parts:
- added C10: 22uF, passive:0402, F.Cu at (112.6, 84.7)
- added C11: 1uF, passive:0402, F.Cu at (112.6, 86.6)
- added C12: 4.7uF, passive:0402, F.Cu at (112.6, 88.5)
- added C13: 1uF, passive:0402, F.Cu at (112.6, 90.4)
- added C14: 1uF, passive:0402, F.Cu at (112.6, 92.3)
- added C7: 2.2uF, passive:0402, F.Cu at (109.8, 92.3)
- added C8: 1uF, passive:0402, F.Cu at (118.5, 103.0)
- added C9: 4.7uF, passive:0402, F.Cu at (112.6, 82.8)
- added J2: 53261-0271, connector:53261-0271, B.Cu at (126.0, 105.0)
- added R10: 100K, passive:0402, F.Cu at (118.2, 84.7)
- added R6: 27R, passive:0402, F.Cu at (115.4, 90.4)
- added R7: 27R, passive:0402, B.Cu at (109.5, 104.0)
- added R8: 10K, passive:0402, F.Cu at (118.2, 80.9)
- added R9: 10K, passive:0402, F.Cu at (118.2, 82.8)
- added RT1: NTCLE413E2103H400, passive:THT2, F.Cu at (123.0, 109.0)
- added S1: TL3365AF180QG, connector:TL3365AF180QG, B.Cu at (103.0, 105.0)
- C1: value 4.7uF -> 22uF; footprint passive:0603 -> passive:0402
- C2: value 1uF -> 22uF
- C3: footprint passive:0603 -> passive:0402
- C4: value 3300pF -> 22uF
- C5: value 4.7uF -> 3300pF; footprint passive:0603 -> passive:0402
- C6: value 22uF -> 2.2uF; footprint passive:0603 -> passive:0402
- R1, R2: value 5K -> 0R
- R3: value 27R -> 0R
- R4: value 27R -> 5K
- R5: value 0R -> 5K
- moved C2 62.3 mm to (109.8, 82.8)
- moved C4 60.9 mm to (109.8, 86.6)
- moved C3 60.5 mm to (109.8, 84.7)
- moved C6 59.1 mm to (109.8, 90.4)
- moved C5 59.1 mm to (109.8, 88.5)
- moved R5 57.3 mm to (115.4, 88.5)
- moved R4 50.6 mm to (115.4, 86.6)
- moved R1 50.1 mm to (115.4, 80.9)
- moved R2 50.1 mm to (115.4, 82.8)
- moved R3 50.1 mm to (115.4, 84.7)
- moved L1 45.5 mm to (115.2, 108.0)
- moved C1 44.7 mm to (122.5, 93.0)
- moved U1 38.7 mm to (115.0, 105.0)
- moved J1 33.8 mm to (102.0, 105.0)
Connections:
- C1 pad 1: /CHGIN -> /SSB1
- C2 pad 1: /VL -> /SSB0
- C3 pad 1: Net-(U1-IN_SBB) -> /SSB2
- C4 pad 1: /BST -> Net-(U1-IN_SBB)
- C4 pad 2: /LXB -> GND
- C5 pad 1: GND -> /BST
- C5 pad 2: /BATT -> /LXB
- C6 pad 1: /BATT -> /IN_LDO0
- R1 pad 1: GND -> /SSB0
- R1 pad 2: /USB_CC1 -> /IN_LDO1
- R2 pad 1: GND -> /SSB0
- R2 pad 2: /USB_CC2 -> /IN_LDO0
- R3 pad 1: /MCU_USB_DP -> Net-(U1-IN_SBB)
- R3 pad 2: /USB_DP -> /V_SYS
- R4 pad 1: /MCU_USB_DN -> GND
- R4 pad 2: /USB_DN -> /USB_CC1
- R5 pad 1: Net-(U1-IN_SBB) -> GND
- R5 pad 2: /V_SYS -> /USB_CC2
- U1 pad A1: unconnected-(U1-GPIO1-PadA1) -> /GPIO1
- U1 pad A2: unconnected-(U1-NRST-PadA2) -> /nRST
- U1 pad A4: unconnected-(U1-VIO-PadA4) -> /VIO
- U1 pad A5: unconnected-(U1-LDO1-PadA5) -> /LDO1
- U1 pad A6: unconnected-(U1-IN_LDO1-PadA6) -> /IN_LDO1
- U1 pad B1: unconnected-(U1-GPIO0-PadB1) -> /GPIO0
- U1 pad B2: unconnected-(U1-NIRQ-PadB2) -> /nIRQ
- U1 pad B3: unconnected-(U1-NEN-PadB3) -> /nEN
- U1 pad B5: unconnected-(U1-LDO0-PadB5) -> /LDO0
- U1 pad B6: unconnected-(U1-IN_LDO0-PadB6) -> /IN_LDO0
- U1 pad C1: unconnected-(U1-AMUX-PadC1) -> /AMUX
- U1 pad C2: unconnected-(U1-GPIO2-PadC2) -> /GPIO2
- U1 pad C3: unconnected-(U1-GND-PadC3) -> GND
- U1 pad C4: unconnected-(U1-SBB1-PadC4) -> /SSB1
- U1 pad C6: unconnected-(U1-SBB0-PadC6) -> /SSB0
- U1 pad D1: unconnected-(U1-VL-PadD1) -> /VL
- U1 pad D2: unconnected-(U1-THM-PadD2) -> /THM
- U1 pad D3: unconnected-(U1-TBIAS-PadD3) -> /TBIAS
- U1 pad D4: unconnected-(U1-SBB2-PadD4) -> /SSB2
Other:
- board size 50.8 x 50.8 mm -> 30 x 10 mm

Commit message: layout almost finished
Parts:
- removed C6, C7: 2.2uF, passive:0402
- removed R1, R2, R3: 0R, passive:0402
- added C15: 22uF, passive:0402, F.Cu at (113.0, 107.4)
- C4: footprint passive:0402 -> passive:0603
- R4, R5, R6: moved to B.Cu
- moved R9 32.5 mm to (112.7, 114.9)
- moved R10 28.3 mm to (112.7, 112.5)
- moved R8 28.1 mm to (120.4, 109.0)
- moved C5 25.2 mm to (112.7, 113.6)
- moved C9 24.6 mm to (114.1, 107.4), turned to 90 degrees
- moved C3 22.7 mm to (117.7, 106.0)
- moved C2 22.6 mm to (117.7, 104.0)
- moved C10 22.4 mm to (122.1, 105.0), turned to -90 degrees
- moved C4 21.3 mm to (115.9, 107.0)
- moved R4 21.1 mm to (109.0, 106.7), turned to 180 degrees
- moved C12 17.4 mm to (112.4, 105.9)
- moved R6 16.5 mm to (109.0, 105.6), turned to 180 degrees
- moved C11 16.2 mm to (115.8, 102.5), turned to 90 degrees
- moved R5 16.2 mm to (109.0, 103.4), turned to 180 degrees
- moved C13 14.2 mm to (112.4, 104.6), turned to 180 degrees
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Connections:
- C4 pad 1: Net-(U1-IN_SBB) -> /V_SYS
- U1 pad A6: /IN_LDO1 -> /SSB0
- U1 pad B6: /IN_LDO0 -> /SSB0
- U1 pad E4: Net-(U1-IN_SBB) -> /V_SYS
Routing:
- added copper zone on F.Cu, net /LXA
Other:
- board size 30 x 10 mm -> 30 x 11 mm

Commit message: almost done the PCB
Parts:
- moved R9 12.5 mm to (113.6, 102.5), turned to -90 degrees
- moved RT1 11.2 mm to (111.8, 108.5), turned to 90 degrees
- moved R10 10.1 mm to (112.5, 102.5), turned to 90 degrees
- moved C5 8.04 mm to (118.1, 107.7), turned to -90 degrees
- moved R8 6.96 mm to (113.4, 109.1)
- moved C4 0.15 mm to (115.9, 107.2)
- moved C15 0.15 mm to (113.0, 107.5)
- moved C9 0.15 mm to (114.1, 107.5)
- moved C12 0.10 mm to (112.3, 105.9)
- moved C13 0.10 mm to (112.3, 104.6)
- moved L1 0.10 mm to (116.1, 108.6)
Connections:
- U1 pad A3: unconnected-(U1-SDA-PadA3) -> /SDA
- U1 pad B4: unconnected-(U1-SCL-PadB4) -> /SCL
Routing:
- net /nEN: track 0.00 -> 18.8 mm, vias 0 -> 2
- net /THM: track 0.00 -> 7.03 mm, vias 0 -> 1
- net /V_SYS: track 0.00 -> 5.39 mm, vias 0 -> 3
- net /AMUX: track 0.00 -> 4.13 mm
- net /TBIAS: track 0.00 -> 4.05 mm, vias 0 -> 2
- net /nIRQ: track 0.00 -> 3.81 mm, vias 0 -> 1
- net /GPIO0: track 0.00 -> 3.49 mm
- net /SCL: track 0.00 -> 3.12 mm, vias 0 -> 1
- net /GPIO1: track 0.00 -> 3.00 mm
- net /nRST: track 0.00 -> 2.69 mm, vias 0 -> 2
- net /SDA: track 0.00 -> 2.40 mm, vias 0 -> 1
- net /SSB2: track 0.00 -> 2.25 mm, vias 0 -> 2
- net /VIO: track 0.00 -> 2.20 mm
- net /LDO0: track 0.00 -> 2.19 mm, vias 0 -> 2
- net /SSB1: track 0.00 -> 2.06 mm, vias 0 -> 2
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- added copper zone on F.Cu, net /BATT
- added copper zone on F.Cu, net /CHGIN
- added copper zone on F.Cu, net /LDO1
- added copper zone on In1.Cu, net /LXB
- added copper zone on F.Cu, net /SSB0
- added copper zone on F.Cu, net /VIO
- added copper zone on F.Cu, net /VL
- added copper zone on F.Cu, net /V_SYS
- added copper zone on B.Cu, net GND
- added copper zone on F.Cu, net GND
- added copper zone on In1.Cu, net GND
- added copper zone on In2.Cu, net GND

Commit message: backup
Parts:
- removed R6, R7: 27R, passive:0402
- added J4: ~, connector:Connector_20PIN_5052782033, B.Cu at (114.0, 103.0)
- J2: moved to F.Cu
- moved J2 4.10 mm to (121.9, 105.0), turned to -90 degrees
- moved R4 4.04 mm to (105.0, 106.1), turned to -90 degrees
- moved R5 4.03 mm to (105.0, 103.9), turned to -90 degrees
- moved C10 3.93 mm to (119.2, 107.7)
- moved S1 0.50 mm to (102.5, 105.0), turned to 90 degrees
- moved J1 0.30 mm to (102.6, 105.0)
- moved RT1 0.11 mm to (111.8, 108.6)
- turned R10 to -90 degrees
- turned R9 to 90 degrees
Connections:
- J1 pad A6: /USB_DP -> unconnected-(J1-DP1-PadA6)
- J1 pad A7: /USB_DN -> unconnected-(J1-DN1-PadA7)
Routing:
- net /CHGIN: track 0.00 -> 17.6 mm, vias 0 -> 2
- net /BATT: track 0.26 -> 15.0 mm, vias 0 -> 4
- net GND: track 0.00 -> 12.4 mm, vias 3 -> 21
- net /SSB2: track 2.25 -> 9.72 mm
- net /SSB1: track 2.06 -> 7.62 mm
- net /TBIAS: track 4.05 -> 9.12 mm
- net /SSB0: track 0.20 -> 4.21 mm
- net /LDO0: track 2.19 -> 5.22 mm
- net /BST: track 0.00 -> 3.01 mm, vias 0 -> 2
- net /LDO1: track 0.00 -> 2.99 mm, vias 0 -> 1
- net /nEN: track 18.8 -> 21.5 mm, vias 2 -> 1
- net /USB_CC2: track 0.00 -> 2.62 mm, vias 0 -> 1
- net /USB_CC1: track 0.00 -> 2.42 mm, vias 0 -> 1
- net /SDA: track 2.40 -> 4.45 mm
- net /THM: track 7.03 -> 8.85 mm
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Other:
- board size 30 x 11 mm -> 25 x 11 mm

Commit message: done ;).
Parts:
- removed C11, C8: 1uF, passive:0402
- added C6: 1uF, passive:C_0402, F.Cu at (116.8, 102.5)
- added C7: 1uF, passive:C_0402, F.Cu at (115.8, 102.5)
- added J3: ~, connector:Header_THT_1.27_3P, F.Cu at (110.0, 103.8)
- C1, C10, C12, C13, C14, C15, C2, C3, C5, C9: footprint passive:0402 -> passive:C_0402
- C4: footprint passive:0603 -> passive:C_0603
- L1: footprint passive:2016 -> passive:L_0806
- R10, R4, R5, R8, R9: footprint passive:0402 -> passive:R_0402
- moved C3 2.10 mm to (117.7, 104.0)
- moved J4 1.50 mm to (115.5, 103.1)
- moved S1 1.20 mm to (103.7, 105.0)
- moved C1 1.05 mm to (117.7, 106.0)
- moved C2 1.05 mm to (117.7, 105.0)
- moved R4 1.00 mm to (106.0, 106.1)
- moved R5 1.00 mm to (106.0, 103.9)
- moved J2 0.40 mm to (122.3, 105.0)
- moved RT1 0.31 mm to (111.8, 108.3)
Connections:
- net /USB_CC1 renamed Net-(J1-CC2)
- net /USB_CC2 renamed Net-(J1-CC1)
- C1 pad 1: /SSB1 -> /SSB2
- C2 pad 1: /SSB0 -> /SSB1
- C3 pad 1: /SSB2 -> /SSB0
- J1 pad B6: /USB_DP -> unconnected-(J1-DP2-PadB6)
- J1 pad B7: /USB_DN -> unconnected-(J1-DN2-PadB7)
- U1 pad C2: /GPIO2 -> unconnected-(U1-GPIO2-PadC2)
Routing:
- net GND: track 12.4 -> 2.73 mm, vias 21 -> 37
- net /CHGIN: track 17.6 -> 14.3 mm
- net /GPIO1: track 2.85 -> 4.39 mm, vias 1 -> 0
- net /nEN: track 21.5 -> 20.0 mm
- net Net-(J1-CC1): track 2.62 -> 1.62 mm
- net Net-(J1-CC2): track 2.42 -> 1.42 mm
- net /SCL: track 4.80 -> 4.08 mm
- net /AMUX: track 3.94 -> 4.58 mm, vias 1 -> 0
- net /LDO0: track 5.22 -> 4.58 mm
- net /LDO1: track 2.99 -> 2.43 mm
- net /GPIO0: track 3.60 -> 4.03 mm, vias 1 -> 0
- net /BATT: vias 4 -> 3
- added copper zone on B.Cu, net /CHGIN

Commit message: optimize footprints
Parts:
- J3: value ~ -> M50-3530342
- J4: value ~ -> 5052782033
Changed lines of the file:
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@@
     (fp_circle (center -1.458 -1.258) (end -1.458 -1.158)
       (stroke (width 0.2) (type solid)) (fill none) (layer "F.SilkS"))
-    (fp_line (start -2.406 -2.182) (end 2.407 -2.182)
+    (fp_line (start -1.7 -1.5) (end 1.7 -1.5)
       (stroke (width 0.05) (type solid)) (layer "F.CrtYd"))
-    (fp_line (start -2.406 2.181) (end -2.406 -2.182)
+    (fp_line (start -1.7 1.5) (end -1.7 -1.5)
       (stroke (width 0.05) (type solid)) (layer "F.CrtYd"))
-    (fp_line (start 2.407 -2.182) (end 2.407 2.181)
+    (fp_line (start 1.7 -1.5) (end 1.7 1.5)
       (stroke (width 0.05) (type solid)) (layer "F.CrtYd"))
-    (fp_line (start 2.407 2.181) (end -2.406 2.181)
+    (fp_line (start 1.7 1.5) (end -1.7 1.5)
       (stroke (width 0.05) (type solid)) (layer "F.CrtYd"))
     (fp_line (start -1.394 -1.169) (end 1.394 -1.169)
@@
     (fp_arc (start 0.7 3.4) (mid 0.65 3.45) (end 0.6 3.4)
       (stroke (width 0.1) (type solid)) (layer "F.SilkS"))
-    (fp_line (start -5.225 -3.3) (end -5.225 4.45)
+    (fp_line (start -3.6 -2.6) (end 3.6 -2.6)
+      (stroke (width 0.1) (type default)) (layer "Margin"))
+    (fp_line (start -1.2 1.9) (end -3.6 1.9)
+      (stroke (width 0.1) (type default)) (layer "Margin"))
+    (fp_line (start -1.2 3.4) (end -1.2 1.9)
+      (stroke (width 0.1) (type default)) (layer "Margin"))
+    (fp_line (start 1.2 1.9) (end 1.2 3.4)
+      (stroke (width 0.1) (type default)) (layer "Margin"))
+    (fp_line (start 3.6 1.9) (end 1.2 1.9)
+      (stroke (width 0.1) (type default)) (layer "Margin"))
+    (fp_line (start -3.6 -2.6) (end -3.6 1.9)
       (stroke (width 0.1) (type solid)) (layer "F.CrtYd"))
-    (fp_line (start -5.225 4.45) (end 5.225 4.45)
+    (fp_line (start -1.2 3.4) (end 1.2 3.4)
       (stroke (width 0.1) (type solid)) (layer "F.CrtYd"))
-    (fp_line (start 5.225 -3.3) (end -5.225 -3.3)
-      (stroke (width 0.1) (type solid)) (layer "F.CrtYd"))
-    (fp_line (start 5.225 4.45) (end 5.225 -3.3)
+    (fp_line (start 3.6 1.9) (end 3.6 -2.6)
       (stroke (width 0.1) (type solid)) (layer "F.CrtYd"))
     (fp_line (start -3.625 -2.3) (end -3.625 1.9)
@@
         (effects (font (size 0.8 0.8) (thickness 0.1)))
     )
-    (fp_text value "~" (at 0 1 -90 unlocked) (layer "Cmts.User") hide
+    (fp_text value "M50-3530342" (at 0 1 -90 unlocked) (layer "Cmts.User") hide
         (effects (font (size 0.3 0.3) (thickness 0.05) bold))
     )
@@
         (effects (font (size 0.8 0.8) (thickness 0.1)) (justify mirror))
     )
-    (fp_text value "~" (at 0 -0.8 unlocked) (layer "Cmts.User")
+    (fp_text value "5052782033" (at 0 -0.8 unlocked) (layer "Cmts.User")
         (effects (font (size 0.3 0.3) (thickness 0.05)))
     )
@@
     (fp_line (start 2.1 0.5) (end 2.1 -0.5)
       (stroke (width 0.1) (type solid)) (layer "B.SilkS"))
-    (fp_line (start -4.2 -2.6) (end -4.2 2.6)
+    (fp_line (start -2.9 -1.8) (end -2.9 1.8)
       (stroke (width 0.1) (type solid)) (layer "B.CrtYd"))
-    (fp_line (start -4.2 2.6) (end 3.75 2.6)
+    (fp_line (start -2.9 1.8) (end 2.9 1.8)
       (stroke (width 0.1) (type solid)) (layer "B.CrtYd"))
-    (fp_line (start 3.75 -2.6) (end -4.2 -2.6)
+    (fp_line (start 2.9 -1.8) (end -2.9 -1.8)
       (stroke (width 0.1) (type solid)) (layer "B.CrtYd"))
-    (fp_line (start 3.75 2.6) (end 3.75 -2.6)
+    (fp_line (start 2.9 1.8) (end 2.9 -1.8)
       (stroke (width 0.1) (type solid)) (layer "B.CrtYd"))
     (fp_line (start -2.1 -1.6) (end -2.1 1.6)
