File: elastic_power_module.kicad_pcb (KiCad board)
At the start: 4 copper layers, 25 x 11 mm, 26 parts, among them J1 USB4105GFA060, J2 53261-0271, U1 MAX77654AENV+T

Commit message: update pcb file
Parts:
- J3: value ~ -> M50-3530342
- J4: value ~ -> 5052782033
Changed lines of the file:
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@@
         (effects (font (size 0.8 0.8) (thickness 0.1)))
     )
-    (fp_text value "~" (at 0 1 -90 unlocked) (layer "Cmts.User") hide
+    (fp_text value "M50-3530342" (at 0 1 -90 unlocked) (layer "Cmts.User") hide
         (effects (font (size 0.3 0.3) (thickness 0.05) bold))
     )
@@
         (effects (font (size 0.8 0.8) (thickness 0.1)) (justify mirror))
     )
-    (fp_text value "~" (at 0 -0.8 unlocked) (layer "Cmts.User")
-        (effects (font (size 0.3 0.3) (thickness 0.05)))
-    )
+    (fp_text value "5052782033" (at 0 -0.8 unlocked) (layer "Cmts.User")
+        (effects (font (size 0.3 0.3) (thickness 0.05)))
+    )
